File: STM32F401/STM32F4XX.sch (KiCad schematic (older format))
At the start: 33 parts, among them J1 DEBUG UART, J2 Conn_02x16_Counter_Clockwise, J3 USB_B_Mini, J4 Conn_02x16_Counter_Clockwise, J5 JTAG SWDIO SWCLK, SW1 ~RESET, U1 STM32F401RCT6, U2 LM1117-3.3, Y1 8MHz

Commit message: Added KiCAD loAdded KiCAD logo on back silkscreen
Parts:
- added LOGO2: designed with KiCAD, Symbol:KiCad-Logo2_6mm_SilkScreen, symbol AmigaComponents:LOGO
- renumbered LOGO2 to LOGO1
Changed lines of the file:
@@
 Sheet 1 1
 Title "GENERIC STM32F401 MODULE"
-Date "2022-01-11"
-Rev "0.1"
+Date "2022-02-05"
+Rev "0.2"
 Comp "RetroBit Lab"
 Comment1 ""
@@
 $EndComp
 $Comp
+L AmigaComponents:LOGO LOGO1
+U 1 1 61DE4C48
+P 7270 6060
+F 0 "LOGO1" H 7295 6113 59  0000 L CNN
+F 1 "OSH" H 7295 6008 59  0000 L CNN
+F 2 "Symbol:OSHW-Logo_11.4x12mm_SilkScreen" H 7270 6060 59  0001 C CNN
+F 3 "" H 7270 6060 59  0001 C CNN
+	1    7270 6060
+	1    0    0    -1
+$EndComp
+$Comp
 L AmigaComponents:LOGO LOGO2
-U 1 1 61DE4C48
-P 7405 5895
-F 0 "LOGO2" H 7430 5948 59  0000 L CNN
-F 1 "OSH" H 7430 5843 59  0000 L CNN
-F 2 "Symbol:OSHW-Logo_11.4x12mm_SilkScreen" H 7405 5895 59  0001 C CNN
-F 3 "" H 7405 5895 59  0001 C CNN
-	1    7405 5895
-	1    0    0    -1
-$EndComp
+U 1 1 62003E98
+P 7705 6105
+F 0 "LOGO2" H 7745 6210 59  0000 L CNN
+F 1 "designed with KiCAD" H 7735 6120 59  0000 L CNN
+F 2 "Symbol:KiCad-Logo2_6mm_SilkScreen" H 7705 6105 59  0001 C CNN
+F 3 "" H 7705 6105 59  0001 C CNN
+	1    7705 6105
+	1    0    0    -1
+$EndComp

Commit message: Added RESET switch
Parts:
- SW1: LCSC (none) -> C318911
Changed lines of the file:
@@
 F 2 "RetroBitLab:SW_SPST_FSMSM_3D" H 4130 2555 50  0001 C CNN
 F 3 "~" H 4130 2555 50  0001 C CNN
+F 4 "C318911" V 4130 2355 50  0001 C CNN "LCSC"
 	1    4130 2355
 	0    -1   -1   0

Commit message: Updated footprint for RESET switch. It will a 7.3x3.9x2.5 mm like a Wuerth 434121025816
Parts:
- SW1: footprint RetroBitLab:SW_SPST_FSMSM_3D -> RetroBitLab:SPST-7.3x3.9x2.5-WUERTH-434121025816
Changed lines of the file:
@@
 F 0 "SW1" V 4255 2610 50  0000 R CNN
 F 1 "~RESET" V 4130 2765 50  0000 R CNN
-F 2 "RetroBitLab:SW_SPST_FSMSM_3D" H 4130 2555 50  0001 C CNN
+F 2 "RetroBitLab:SPST-7.3x3.9x2.5-WUERTH-434121025816" H 4130 2555 50  0001 C CNN
 F 3 "~" H 4130 2555 50  0001 C CNN
 F 4 "C318911" V 4130 2355 50  0001 C CNN "LCSC"
